File: modulo-ergo42/modulo-ergo42.sch (KiCad schematic (older format))
At the start: 38 parts, among them J1 AudioJack4_Ground, J2 AudioJack4_Ground, J3 AudioJack4_Ground, J4 AudioJack4_Ground, SW1 SW_Push, SW10 SW_Push, SW11 SW_Push, SW12 SW_Push, SW13 SW_Push, SW14 SW_Push, SW15 SW_Push, SW16 SW_Push, SW17 SW_Push, SW18 SW_Push, SW19 SW_Push, SW2 SW_Push, SW20 SW_Push, SW21 SW_Push, SW22 SW_Push, SW23 SW_Push, SW24 SW_Push, SW25 SW_Push, SW26 SW_Push, SW27 SW_Push, SW28 SW_Push, SW29 SW_DIP_x02, SW3 SW_Push, SW4 SW_Push, SW5 SW_Push, SW6 SW_Push, SW7 SW_Push, SW8 SW_Push, SW9 SW_Push, U1 TCA9555PWR, U2 TCA9555PWR

Commit message: Update schematics for beta
Parts:
- removed J1, J2, J3, J4: AudioJack4_Ground, library:TRRS_SMD_PJ320, symbol Connector:AudioJack4_Ground
- added C1, C2: 100 p, Capacitor_SMD:C_0603_1608Metric, symbol Device:C_Small
- added C3: 1 u, Capacitor_SMD:C_0603_1608Metric, symbol Device:C_Small
- added J1, J2, J3, J4: AudioJack4, library:TRRS_SMD_PJ320, symbol Connector:AudioJack4
- R2, R3: value 10 kΩ -> 1 M
Connections:
- net GND: now also C1.2, C2.2, C3.2, J1.S, J2.S, J3.S, J4.S
- net INT: now also J3.R1, J4.R1
- net R1C1: now also U1.4 (P00); no longer U1.7 (P03)
- net R1C2: now also U1.5 (P01); no longer U1.11 (P07)
- net R1C3: now also U1.6 (P02); no longer U1.13 (P10)
- net R1C4: now also U1.7 (P03); no longer U1.17 (P14)
- net R1C5: now also U1.8 (P04); no longer U2.7 (P03)
- net R1C6: now also U1.9 (P05); no longer U2.11 (P07)
- net R1C7: now also U1.10 (P06); no longer U2.13 (P10)
- net R2C1: now also U1.19 (P16); no longer U1.6 (P02)
- net R2C2: now also U1.18 (P15); no longer U1.10 (P06)
- net R2C3: now also U1.17 (P14); no longer U1.14 (P11)
- net R2C4: now also U1.16 (P13); no longer U1.18 (P15)
- net R2C5: now also U1.15 (P12); no longer U2.6 (P02)
- net R2C6: now also U1.14 (P11); no longer U2.10 (P06)
- net R2C7: now also U1.13 (P10); no longer U2.14 (P11)
- net R3C1: now also U2.4 (P00); no longer U1.5 (P01)
- net R3C2: now also U2.5 (P01); no longer U1.9 (P05)
- net R3C3: now also U2.6 (P02); no longer U1.15 (P12)
- net R3C4: now also U2.7 (P03); no longer U1.19 (P16)
- net R3C5: now also U2.8 (P04); no longer U2.5 (P01)
- net R3C7: now also U2.10 (P06); no longer U2.15 (P12)
- net R4C1: now also U2.19 (P16); no longer U1.4 (P00)
- net R4C2: now also U2.18 (P15); no longer U1.8 (P04)
- net R4C3: now also U2.17 (P14); no longer U1.16 (P13)
- net R4C4: now also U2.16 (P13); no longer U1.20 (P17)
- net R4C5: now also U2.15 (P12); no longer U2.4 (P00)
- net R4C6: now also U2.14 (P11); no longer U2.8 (P04)
- net R4C7: now also U2.13 (P10); no longer U2.16 (P13)
- net SCL: now also J1.R1, J2.R1
- net SDA: now also J1.R2, J2.R2
- net VCC: now also C1.1, C2.1, C3.1, J1.T, J2.T, J3.T, J4.T
Changed lines of the file:
@@
-$EndComp
-$Comp
-L Connector:AudioJack4_Ground J1
-U 1 1 5BC2FF07
-P 1000 2200
-F 0 "J1" H 966 2542 50  0000 C CNN
-F 1 "AudioJack4_Ground" H 966 2451 50  0000 C CNN
-F 2 "library:TRRS_SMD_PJ320" H 1000 2200 50  0001 C CNN
-F 3 "~" H 1000 2200 50  0001 C CNN
-	1    1000 2200
-	1    0    0    -1
-$EndComp
-$Comp
-L Connector:AudioJack4_Ground J2
-U 1 1 5BC30075
-P 2000 2200
-F 0 "J2" H 1966 2542 50  0000 C CNN
-F 1 "AudioJack4_Ground" H 1966 2451 50  0000 C CNN
-F 2 "library:TRRS_SMD_PJ320" H 2000 2200 50  0001 C CNN
-F 3 "~" H 2000 2200 50  0001 C CNN
-	1    2000 2200
-	1    0    0    -1
 $EndComp
 $Comp
@@
 	0    -1   -1   0
 $EndComp
+Text GLabel 1200 2300 2    50   Input ~ 0
+SCL
 Text GLabel 1200 2200 2    50   Input ~ 0
+SDA
+Text GLabel 2200 2300 2    50   Input ~ 0
 SCL
-Text GLabel 1200 2300 2    50   Input ~ 0
-SDA
 Text GLabel 2200 2200 2    50   Input ~ 0
-SCL
-Text GLabel 2200 2300 2    50   Input ~ 0
 SDA
 $Comp
@@
 	1    0    0    -1
 $EndComp
-Text GLabel 1450 4200 0    50   Input ~ 0
+Text GLabel 1250 4200 0    50   Input ~ 0
 3V3
-Text GLabel 1450 6500 0    50   Input ~ 0
+Text GLabel 1250 6500 0    50   Input ~ 0
 3V3
-$Comp
-L Connector:AudioJack4_Ground J3
-U 1 1 5BC32F04
-P 3000 2200
-F 0 "J3" H 2966 2542 50  0000 C CNN
-F 1 "AudioJack4_Ground" H 2966 2451 50  0000 C CNN
-F 2 "library:TRRS_SMD_PJ320" H 3000 2200 50  0001 C CNN
-F 3 "~" H 3000 2200 50  0001 C CNN
-	1    3000 2200
-	1    0    0    -1
-$EndComp
 $Comp
 L power:GND #PWR010
@@
 P 9600 1250
 F 0 "R2" H 9530 1296 50  0000 R CNN
-F 1 "10 kΩ" H 9530 1205 50  0000 R CNN
+F 1 "1 M" H 9530 1205 50  0000 R CNN
 F 2 "Resistor_SMD:R_0603_1608Metric" V 9530 1250 50  0001 C CNN
 F 3 "~" H 9600 1250 50  0001 C CNN
@@
 P 10000 1250
 F 0 "R3" H 9930 1296 50  0000 R CNN
-F 1 "10 kΩ" H 9930 1205 50  0000 R CNN
+F 1 "1 M" H 9930 1205 50  0000 R CNN
 F 2 "Resistor_SMD:R_0603_1608Metric" V 9930 1250 50  0001 C CNN
 F 3 "~" H 10000 1250 50  0001 C CNN
@@
 	9900 1450 9900 1600
 Connection ~ 9900 1600
-NoConn ~ 3050 5800
-NoConn ~ 3250 5800
-NoConn ~ 3350 5800
-NoConn ~ 3150 5800
+Text GLabel 1750 3500 1    50   Input ~ 0
+R1C1
+Text GLabel 1850 3500 1    50   Input ~ 0
+R1C2
+Text GLabel 3250 3500 1    50   Input ~ 0
+R2C1
+Text GLabel 1750 5800 1    50   Input ~ 0
+R3C1
+Text GLabel 3250 5800 1    50   Input ~ 0
+R4C1
+Text GLabel 3150 3500 1    50   Input ~ 0
+R2C2
+Text GLabel 1850 5800 1    50   Input ~ 0
+R3C2
+Text GLabel 3150 5800 1    50   Input ~ 0
+R4C2
+Text GLabel 1950 3500 1    50   Input ~ 0
+R1C3
+Text GLabel 3050 3500 1    50   Input ~ 0
+R2C3
+Text GLabel 1950 5800 1    50   Input ~ 0
+R3C3
+Text GLabel 3050 5800 1    50   Input ~ 0
+R4C3
 Text GLabel 2050 3500 1    50   Input ~ 0
-R1C1
-Text GLabel 2450 3500 1    50   Input ~ 0
-R1C2
-Text GLabel 1950 3500 1    50   Input ~ 0
-R2C1
-Text GLabel 1850 3500 1    50   Input ~ 0
-R3C1
-Text GLabel 1750 3500 1    50   Input ~ 0
-R4C1
-Text GLabel 2350 3500 1    50   Input ~ 0
-R2C2
+R1C4
+Text GLabel 2950 3500 1    50   Input ~ 0
+R2C4
+Text GLabel 2050 5800 1    50   Input ~ 0
+R3C4
+Text GLabel 2950 5800 1    50   Input ~ 0
+R4C4
+Text GLabel 2150 3500 1    50   Input ~ 0
+R1C5
+Text GLabel 2850 3500 1    50   Input ~ 0
+R2C5
+Text GLabel 2150 5800 1    50   Input ~ 0
+R3C5
+Text GLabel 2850 5800 1    50   Input ~ 0
+R4C5
 Text GLabel 2250 3500 1    50   Input ~ 0
-R3C2
-Text GLabel 2150 3500 1    50   Input ~ 0
-R4C2
-Text GLabel 2650 3500 1    50   Input ~ 0
-R1C3
+R1C6
 Text GLabel 2750 3500 1    50   Input ~ 0
-R2C3
-Text GLabel 2850 3500 1    50   Input ~ 0
-R3C3
-Text GLabel 2950 3500 1    50   Input ~ 0
-R4C3
-Text GLabel 3050 3500 1    50   Input ~ 0
-R1C4
-Text GLabel 3150 3500 1    50   Input ~ 0
-R2C4
-Text GLabel 3250 3500 1    50   Input ~ 0
-R3C4
-Text GLabel 3350 3500 1    50   Input ~ 0
-R4C4
-Text GLabel 2050 5800 1    50   Input ~ 0
-R1C5
-Text GLabel 1950 5800 1    50   Input ~ 0
-R2C5
-Text GLabel 1850 5800 1    50   Input ~ 0
-R3C5
-Text GLabel 1750 5800 1    50   Input ~ 0
-R4C5
-Text GLabel 2450 5800 1    50   Input ~ 0
-R1C6
-Text GLabel 2350 5800 1    50   Input ~ 0
 R2C6
 Text GLabel 2250 5800 1    50   Input ~ 0
 R3C6
-Text GLabel 2150 5800 1    50   Input ~ 0
+Text GLabel 2750 5800 1    50   Input ~ 0
 R4C6
+Text GLabel 2350 3500 1    50   Input ~ 0
+R1C7
+Text GLabel 2650 3500 1    50   Input ~ 0
+R2C7
+Text GLabel 2350 5800 1    50   Input ~ 0
+R3C7
 Text GLabel 2650 5800 1    50   Input ~ 0
-R1C7
-Text GLabel 2750 5800 1    50   Input ~ 0
-R2C7
-Text GLabel 2850 5800 1    50   Input ~ 0
-R3C7
-Text GLabel 2950 5800 1    50   Input ~ 0
 R4C7
 $Comp
@@
 3V3
 $Comp
-L Connector:AudioJack4_Ground J4
-U 1 1 5BC43221
-P 4000 2200
-F 0 "J4" H 3966 2542 50  0000 C CNN
-F 1 "AudioJack4_Ground" H 3966 2451 50  0000 C CNN
-F 2 "library:TRRS_SMD_PJ320" H 4000 2200 50  0001 C CNN
-F 3 "~" H 4000 2200 50  0001 C CNN
-	1    4000 2200
-	1    0    0    -1
-$EndComp
-$Comp
 L power:GND #PWR042
 U 1 1 5BC4348C
@@
 	1    0    0    -1
 $EndComp
+$Comp
+L Connector:AudioJack4 J1
+U 1 1 5C165A23
+P 1000 2200
+F 0 "J1" H 955 2525 50  0000 C CNN
+F 1 "AudioJack4" H 955 2434 50  0000 C CNN
+F 2 "library:TRRS_SMD_PJ320" H 1000 2200 50  0001 C CNN
+F 3 "~" H 1000 2200 50  0001 C CNN
+	1    1000 2200
+	1    0    0    -1
+$EndComp
+$Comp
+L Connector:AudioJack4 J2
+U 1 1 5C165B24
+P 2000 2200
+F 0 "J2" H 1955 2525 50  0000 C CNN
+F 1 "AudioJack4" H 1955 2434 50  0000 C CNN
+F 2 "library:TRRS_SMD_PJ320" H 2000 2200 50  0001 C CNN
+F 3 "~" H 2000 2200 50  0001 C CNN
+	1    2000 2200
+	1    0    0    -1
+$EndComp
+$Comp
+L Connector:AudioJack4 J3
+U 1 1 5C165BD8
+P 3000 2200
+F 0 "J3" H 2955 2525 50  0000 C CNN
+F 1 "AudioJack4" H 2955 2434 50  0000 C CNN
+F 2 "library:TRRS_SMD_PJ320" H 3000 2200 50  0001 C CNN
+F 3 "~" H 3000 2200 50  0001 C CNN
+	1    3000 2200
+	1    0    0    -1
+$EndComp
+$Comp
+L Connector:AudioJack4 J4
+U 1 1 5C165C87
+P 4000 2200
+F 0 "J4" H 3955 2525 50  0000 C CNN
+F 1 "AudioJack4" H 3955 2434 50  0000 C CNN
+F 2 "library:TRRS_SMD_PJ320" H 4000 2200 50  0001 C CNN
+F 3 "~" H 4000 2200 50  0001 C CNN
+	1    4000 2200
+	1    0    0    -1
+$EndComp
+NoConn ~ 2450 3500
+NoConn ~ 3350 3500
+NoConn ~ 3350 5800
+NoConn ~ 2450 5800
+Wire Wire Line
+	1250 4200 1450 4200
+Wire Wire Line
+	1450 6500 1250 6500
+$Comp
+L power:GND #PWR043
+U 1 1 5C16BF77
+P 1250 4400
+F 0 "#PWR043" H 1250 4150 50  0001 C CNN
+F 1 "GND" H 1255 4227 50  0000 C CNN
+F 2 "" H 1250 4400 50  0001 C CNN
+F 3 "" H 1250 4400 50  0001 C CNN
+	1    1250 4400
+	1    0    0    -1
+$EndComp
+$Comp
+L Device:C_Small C1
+U 1 1 5C16C42D
+P 1250 4300
+F 0 "C1" H 1342 4346 50  0000 L CNN
+F 1 "100 p" H 1342 4255 50  0000 L CNN
+F 2 "Capacitor_SMD:C_0603_1608Metric" H 1250 4300 50  0001 C CNN
+F 3 "~" H 1250 4300 50  0001 C CNN
+	1    1250 4300
+	1    0    0    -1
+$EndComp
+$Comp
+L power:GND #PWR044
+U 1 1 5C16C87E
+P 1250 6700
+F 0 "#PWR044" H 1250 6450 50  0001 C CNN
+F 1 "GND" H 1255 6527 50  0000 C CNN
+F 2 "" H 1250 6700 50  0001 C CNN
+F 3 "" H 1250 6700 50  0001 C CNN
+	1    1250 6700
+	1    0    0    -1
+$EndComp
+$Comp
+L Device:C_Small C2
+U 1 1 5C16C884
+P 1250 6600
+F 0 "C2" H 1342 6646 50  0000 L CNN
+F 1 "100 p" H 1342 6555 50  0000 L CNN
+F 2 "Capacitor_SMD:C_0603_1608Metric" H 1250 6600 50  0001 C CNN
+F 3 "~" H 1250 6600 50  0001 C CNN
+	1    1250 6600
+	1    0    0    -1
+$EndComp
+Text GLabel 2650 1050 1    50   Input ~ 0
+3V3
+$Comp
+L Device:C_Small C3
+U 1 1 5C16CE41
+P 2650 1150
+F 0 "C3" H 2742 1196 50  0000 L CNN
+F 1 "1 u" H 2742 1105 50  0000 L CNN
+F 2 "Capacitor_SMD:C_0603_1608Metric" H 2650 1150 50  0001 C CNN
+F 3 "~" H 2650 1150 50  0001 C CNN
+	1    2650 1150
+	1    0    0    -1
+$EndComp
+$Comp
+L power:GND #PWR045
+U 1 1 5C16D074
+P 2650 1250
+F 0 "#PWR045" H 2650 1000 50  0001 C CNN
+F 1 "GND" H 2655 1077 50  0000 C CNN
+F 2 "" H 2650 1250 50  0001 C CNN
+F 3 "" H 2650 1250 50  0001 C CNN
+	1    2650 1250
+	1    0    0    -1
+$EndComp

Commit message: Implement Beta-1
Parts:
- added C4: 1 u, Capacitor_SMD:C_0603_1608Metric, symbol Device:C_Small
Connections:
- net GND: now also C4.2
- net VCC: now also C4.1
Other:
- moved on the sheet: C3
Changed lines of the file:
@@
 L Device:C_Small C3
 U 1 1 5C16CE41
-P 2650 1150
-F 0 "C3" H 2742 1196 50  0000 L CNN
-F 1 "1 u" H 2742 1105 50  0000 L CNN
-F 2 "Capacitor_SMD:C_0603_1608Metric" H 2650 1150 50  0001 C CNN
-F 3 "~" H 2650 1150 50  0001 C CNN
-	1    2650 1150
+P 2650 1250
+F 0 "C3" H 2742 1296 50  0000 L CNN
+F 1 "1 u" H 2742 1205 50  0000 L CNN
+F 2 "Capacitor_SMD:C_0603_1608Metric" H 2650 1250 50  0001 C CNN
+F 3 "~" H 2650 1250 50  0001 C CNN
+	1    2650 1250
 	1    0    0    -1
 $EndComp
@@
 L power:GND #PWR045
 U 1 1 5C16D074
-P 2650 1250
-F 0 "#PWR045" H 2650 1000 50  0001 C CNN
-F 1 "GND" H 2655 1077 50  0000 C CNN
-F 2 "" H 2650 1250 50  0001 C CNN
-F 3 "" H 2650 1250 50  0001 C CNN
-	1    2650 1250
+P 2650 1450
+F 0 "#PWR045" H 2650 1200 50  0001 C CNN
+F 1 "GND" H 2655 1277 50  0000 C CNN
+F 2 "" H 2650 1450 50  0001 C CNN
+F 3 "" H 2650 1450 50  0001 C CNN
+	1    2650 1450
 	1    0    0    -1
 $EndComp
+Wire Wire Line
+	2650 1050 2650 1150
+Wire Wire Line
+	2650 1350 2650 1450
+$Comp
+L Device:C_Small C4
+U 1 1 5C175AF9
+P 3050 1250
+F 0 "C4" H 3142 1296 50  0000 L CNN
+F 1 "1 u" H 3142 1205 50  0000 L CNN
+F 2 "Capacitor_SMD:C_0603_1608Metric" H 3050 1250 50  0001 C CNN
+F 3 "~" H 3050 1250 50  0001 C CNN
+	1    3050 1250
+	1    0    0    -1
+$EndComp
+Wire Wire Line
+	2650 1150 3050 1150
+Connection ~ 2650 1150
+Wire Wire Line
+	3050 1350 2650 1350
+Connection ~ 2650 1350
 $EndSCHEMATC

Commit message: Fix some label
Parts:
- C1, C2: value 100 p -> 100 nF
- C3, C4: value 1 u -> 1 uF
- R2, R3: value 1 M -> 1 MΩ
Changed lines of the file:
@@
 P 9600 1250
 F 0 "R2" H 9530 1296 50  0000 R CNN
-F 1 "1 M" H 9530 1205 50  0000 R CNN
+F 1 "1 MΩ" H 9530 1205 50  0000 R CNN
 F 2 "Resistor_SMD:R_0603_1608Metric" V 9530 1250 50  0001 C CNN
 F 3 "~" H 9600 1250 50  0001 C CNN
@@
 P 10000 1250
 F 0 "R3" H 9930 1296 50  0000 R CNN
-F 1 "1 M" H 9930 1205 50  0000 R CNN
+F 1 "1 MΩ" H 9930 1205 50  0000 R CNN
 F 2 "Resistor_SMD:R_0603_1608Metric" V 9930 1250 50  0001 C CNN
 F 3 "~" H 10000 1250 50  0001 C CNN
@@
 P 1250 4300
 F 0 "C1" H 1342 4346 50  0000 L CNN
-F 1 "100 p" H 1342 4255 50  0000 L CNN
+F 1 "100 nF" H 1342 4255 50  0000 L CNN
 F 2 "Capacitor_SMD:C_0603_1608Metric" H 1250 4300 50  0001 C CNN
 F 3 "~" H 1250 4300 50  0001 C CNN
@@
 P 1250 6600
 F 0 "C2" H 1342 6646 50  0000 L CNN
-F 1 "100 p" H 1342 6555 50  0000 L CNN
+F 1 "100 nF" H 1342 6555 50  0000 L CNN
 F 2 "Capacitor_SMD:C_0603_1608Metric" H 1250 6600 50  0001 C CNN
 F 3 "~" H 1250 6600 50  0001 C CNN
@@
 P 2650 1250
 F 0 "C3" H 2742 1296 50  0000 L CNN
-F 1 "1 u" H 2742 1205 50  0000 L CNN
+F 1 "1 uF" H 2742 1205 50  0000 L CNN
 F 2 "Capacitor_SMD:C_0603_1608Metric" H 2650 1250 50  0001 C CNN
 F 3 "~" H 2650 1250 50  0001 C CNN
@@
 P 3050 1250
 F 0 "C4" H 3142 1296 50  0000 L CNN
-F 1 "1 u" H 3142 1205 50  0000 L CNN
+F 1 "1 uF" H 3142 1205 50  0000 L CNN
 F 2 "Capacitor_SMD:C_0603_1608Metric" H 3050 1250 50  0001 C CNN
 F 3 "~" H 3050 1250 50  0001 C CNN
